File: kicad/tms unit2/tms unit2.kicad_pcb (KiCad board)
At the start: 2 copper layers, 17 parts, among them J1 USB_C_Receptacle_PowerOnly_6P, SW1 NEXT, SW2 CALL_AGAIN, SW3 RESET_QUEUE, U1 ESP32-WROOM-32, U2 AMS1117-3.3

Commit message: improvised  on some aspects
Parts:
- moved J1 78.1 mm to (221.5, 108.5), turned to 90 degrees
- moved SW1 36.0 mm to (190.5, 107.8)
- moved SW3 35.5 mm to (190.5, 122.9)
- moved SW2 14.5 mm to (190.5, 93.0)
- moved C1 7.57 mm to (137.9, 115.8)
- moved C2 7.57 mm to (137.9, 118.8)
- moved C3 7.57 mm to (137.9, 121.8)
- moved C4 7.57 mm to (137.9, 124.8)
- moved C_DB1 7.57 mm to (137.9, 127.8)
- moved C_DB2 7.57 mm to (137.9, 130.8)
- moved R1 7.57 mm to (142.4, 115.8)
- moved R2 7.57 mm to (142.4, 118.7)
- moved R3 7.57 mm to (142.4, 121.7)
- moved R4 7.57 mm to (142.4, 124.6)
- moved U1 7.57 mm to (160.2, 103.2)
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Changed lines of the file:
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@@
 	(footprint "Capacitor_SMD:C_0805_2012Metric"
 		(layer "F.Cu")
-		(at 131.225 118.325)
+		(at 137.95 121.81)
 		(descr "Capacitor SMD 0805 (2012 Metric), square (rectangular) end terminal, IPC-7351 nominal, (Body size source: IPC-SM-782 page 76, https://www.pcb-3d.com/wordpress/wp-content/uploads/ipc-sm-782a_amendment_1_and_2.pdf, https://docs.google.com/spreadsheets/d/1BsfQQcO9C6DZCsRaXUlFlo91Tg2WpOkGARC1WS5S8t0/edit?usp=sharing)")
 		(tags "capacitor")
@@
 	(footprint "Package_TO_SOT_SMD:SOT-223-3_TabPin2"
 		(layer "F.Cu")
-		(at 142.785 124.3)
+		(at 149.51 127.785)
 		(descr "module CMS SOT223 4 pins")
 		(tags "CMS SOT")
@@
 	(footprint "Button_Switch_SMD:SW_SPST_PTS645Sx43SMTR92"
 		(layer "F.Cu")
-		(at 183.625 80.275)
+		(at 190.5 93)
 		(descr "Tactile switch, 6x6 mm, H4.3 mm, gullwing terminals, https://www.ckswitches.com/media/1471/pts645.pdf")
 		(tags "SPST Button Switch CK C&K")
@@
 		)
 		(property "Value" "CALL_AGAIN"
-			(at 0 4.15 0)
+			(at -10.827459 9.403219 0)
 			(layer "F.Fab")
 			(effects
@@
 	(footprint "Capacitor_SMD:C_0805_2012Metric"
 		(layer "F.Cu")
-		(at 131.225 112.305)
+		(at 137.95 115.79)
 		(descr "Capacitor SMD 0805 (2012 Metric), square (rectangular) end terminal, IPC-7351 nominal, (Body size source: IPC-SM-782 page 76, https://www.pcb-3d.com/wordpress/wp-content/uploads/ipc-sm-782a_amendment_1_and_2.pdf, https://docs.google.com/spreadsheets/d/1BsfQQcO9C6DZCsRaXUlFlo91Tg2WpOkGARC1WS5S8t0/edit?usp=sharing)")
 		(tags "capacitor")
@@
 	(footprint "Button_Switch_SMD:SW_SPST_PTS645Sx43SMTR92"
 		(layer "F.Cu")
-		(at 183.625 72.425)
+		(at 190.52 107.75)
 		(descr "Tactile switch, 6x6 mm, H4.3 mm, gullwing terminals, https://www.ckswitches.com/media/1471/pts645.pdf")
 		(tags "SPST Button Switch CK C&K")
@@
 		)
 		(property "Value" "NEXT"
-			(at 0 4.15 0)
+			(at -10.827459 9.403219 0)
 			(layer "F.Fab")
 			(effects
@@
 	(footprint "RF_Module:ESP32-WROOM-32"
 		(layer "F.Cu")
-		(at 153.525 99.765)
+		(at 160.25 103.25)
 		(descr "Single 2.4 GHz Wi-Fi and Bluetooth combo chip https://www.espressif.com/sites/default/files/documentation/esp32-wroom-32_datasheet_en.pdf")
 		(tags "Single 2.4 GHz Wi-Fi and Bluetooth combo  chip")
@@
 			(polygon
 				(pts
-					(xy 129.525 89.965) (xy 177.525 89.965) (xy 177.525 69.025) (xy 129.525 69.025)
+					(xy 136.25 93.45) (xy 184.25 93.45) (xy 184.25 72.51) (xy 136.25 72.51)
 				)
 			)
@@
 	(footprint "Resistor_SMD:R_0805_2012Metric"
 		(layer "F.Cu")
-		(at 135.655 115.225)
+		(at 142.38 118.71)
 		(descr "Resistor SMD 0805 (2012 Metric), square (rectangular) end terminal, IPC-7351 nominal, (Body size source: IPC-SM-782 page 72, https://www.pcb-3d.com/wordpress/wp-content/uploads/ipc-sm-782a_amendment_1_and_2.pdf)")
 		(tags "resistor")
@@
 	(footprint "Capacitor_SMD:C_0805_2012Metric"
 		(layer "F.Cu")
-		(at 131.225 124.345)
+		(at 137.95 127.83)
 		(descr "Capacitor SMD 0805 (2012 Metric), square (rectangular) end terminal, IPC-7351 nominal, (Body size source: IPC-SM-782 page 76, https://www.pcb-3d.com/wordpress/wp-content/uploads/ipc-sm-782a_amendment_1_and_2.pdf, https://docs.google.com/spreadsheets/d/1BsfQQcO9C6DZCsRaXUlFlo91Tg2WpOkGARC1WS5S8t0/edit?usp=sharing)")
 		(tags "capacitor")
@@
 	(footprint "Button_Switch_SMD:SW_SPST_PTS645Sx43SMTR92"
 		(layer "F.Cu")
-		(at 183.625 88.125)
+		(at 190.52 122.9)
 		(descr "Tactile switch, 6x6 mm, H4.3 mm, gullwing terminals, https://www.ckswitches.com/media/1471/pts645.pdf")
 		(tags "SPST Button Switch CK C&K")
@@
 		)
 		(property "Value" "RESET_QUEUE"
-			(at 0 4.15 0)
+			(at -10.827459 9.403219 0)
 			(layer "F.Fab")
 			(effects
@@
 	(footprint "Capacitor_SMD:C_0805_2012Metric"
 		(layer "F.Cu")
-		(at 131.225 121.335)
+		(at 137.95 124.82)
 		(descr "Capacitor SMD 0805 (2012 Metric), square (rectangular) end terminal, IPC-7351 nominal, (Body size source: IPC-SM-782 page 76, https://www.pcb-3d.com/wordpress/wp-content/uploads/ipc-sm-782a_amendment_1_and_2.pdf, https://docs.google.com/spreadsheets/d/1BsfQQcO9C6DZCsRaXUlFlo91Tg2WpOkGARC1WS5S8t0/edit?usp=sharing)")
 		(tags "capacitor")
@@
 	(footprint "Resistor_SMD:R_0805_2012Metric"
 		(layer "F.Cu")
-		(at 135.655 121.125)
+		(at 142.38 124.61)
 		(descr "Resistor SMD 0805 (2012 Metric), square (rectangular) end terminal, IPC-7351 nominal, (Body size source: IPC-SM-782 page 72, https://www.pcb-3d.com/wordpress/wp-content/uploads/ipc-sm-782a_amendment_1_and_2.pdf)")
 		(tags "resistor")
@@
 	(footprint "Capacitor_SMD:C_0805_2012Metric"
 		(layer "F.Cu")
-		(at 131.225 130.365)
+		(at 137.95 133.85)
 		(descr "Capacitor SMD 0805 (2012 Metric), square (rectangular) end terminal, IPC-7351 nominal, (Body size source: IPC-SM-782 page 76, https://www.pcb-3d.com/wordpress/wp-content/uploads/ipc-sm-782a_amendment_1_and_2.pdf, https://docs.google.com/spreadsheets/d/1BsfQQcO9C6DZCsRaXUlFlo91Tg2WpOkGARC1WS5S8t0/edit?usp=sharing)")
 		(tags "capacitor")
@@
 	(footprint "Capacitor_SMD:C_0805_2012Metric"
 		(layer "F.Cu")
-		(at 131.225 127.355)
+		(at 137.95 130.84)
 		(descr "Capacitor SMD 0805 (2012 Metric), square (rectangular) end terminal, IPC-7351 nominal, (Body size source: IPC-SM-782 page 76, https://www.pcb-3d.com/wordpress/wp-content/uploads/ipc-sm-782a_amendment_1_and_2.pdf, https://docs.google.com/spreadsheets/d/1BsfQQcO9C6DZCsRaXUlFlo91Tg2WpOkGARC1WS5S8t0/edit?usp=sharing)")
 		(tags "capacitor")
@@
 	(footprint "Resistor_SMD:R_0805_2012Metric"
 		(layer "F.Cu")
-		(at 135.655 112.275)
+		(at 142.38 115.76)
 		(descr "Resistor SMD 0805 (2012 Metric), square (rectangular) end terminal, IPC-7351 nominal, (Body size source: IPC-SM-782 page 72, https://www.pcb-3d.com/wordpress/wp-content/uploads/ipc-sm-782a_amendment_1_and_2.pdf)")
 		(tags "resistor")
@@
 	(footprint "Connector_USB:USB_C_Receptacle_GCT_USB4125-xx-x_6P_TopMnt_Horizontal"
 		(layer "F.Cu")
-		(at 143.755 115.675)
+		(at 221.5 108.5 90)
 		(descr "USB Type C Receptacle, GCT, power-only, 6P, top mounted, horizontal, 3A, 1mm stake: https://gct.co/files/drawings/usb4125.pdf")
 		(tags "USB C Type-C receptacle power-only charging-only 6P 6C right angled")
 		(property "Reference" "J1"
-			(at 0 -5.1 0)
+			(at 0 -5.1 90)
 			(unlocked yes)
 			(layer "F.SilkS")
@@
 		)
 		(property "Value" "USB_C_Receptacle_PowerOnly_6P"
-			(at 0 4.725 0)
+			(at 0 4.725 90)
 			(unlocked yes)
 			(layer "F.Fab")
@@
 		)
 		(property "Datasheet" ""
-			(at 0 0 0)
+			(at 0 0 90)
 			(unlocked yes)
 			(layer "F.Fab")
@@
 		)
 		(property "Description" ""
-			(at 0 0 0)
+			(at 0 0 90)
 			(unlocked yes)
 			(layer "F.Fab")
@@
 		(duplicate_pad_numbers_are_jumpers no)
 		(fp_line
-			(start -4.67 -0.25)
-			(end -4.67 -1.95)
+			(start 4.67 -0.25)
+			(end 4.67 -1.95)
 			(stroke
 				(width 0.12)
@@
 		)
 		(fp_line
-			(start 4.67 -0.25)
-			(end 4.67 -1.95)
+			(start -4.67 -0.25)
+			(end -4.67 -1.95)
 			(stroke
 				(width 0.12)
@@
 		)
 		(fp_text user "PCB Edge"
-			(at 0 2.825 0)
+			(at 0 2.825 90)
 			(unlocked yes)
 			(layer "Dwgs.User")
@@
 		)
 		(fp_text user "${REFERENCE}"
-			(at 0 -0.275 0)
+			(at 0 -0.275 90)
 			(unlocked yes)
 			(layer "F.Fab")
@@
 		)
 		(pad "A5" smd roundrect
-			(at -0.5 -3.08)
+			(at -0.5 -3.08 90)
 			(size 0.7 1.2)
 			(layers "F.Cu" "F.Mask" "F.Paste")
@@
 		)
 		(pad "A9" smd roundrect
-			(at 1.52 -3.08 180)
+			(at 1.52 -3.08 270)
 			(size 0.76 1.2)
 			(layers "F.Cu" "F.Mask" "F.Paste")
@@
 		)
 		(pad "A12" smd roundrect
-			(at 2.75 -3.08 180)
+			(at 2.75 -3.08 270)
 			(size 0.8 1.2)
 			(layers "F.Cu" "F.Mask" "F.Paste")
@@
 		)
 		(pad "B5" smd roundrect
-			(at 0.5 -3.08 180)
+			(at 0.5 -3.08 270)
 			(size 0.7 1.2)
 			(layers "F.Cu" "F.Mask" "F.Paste")
@@
 		)
 		(pad "B9" smd roundrect
-			(at -1.52 -3.08)
+			(at -1.52 -3.08 90)
 			(size 0.76 1.2)
 			(layers "F.Cu" "F.Mask" "F.Paste")
@@
 		)
 		(pad "B12" smd roundrect
-			(at -2.75 -3.08)
+			(at -2.75 -3.08 90)
 			(size 0.8 1.2)
 			(layers "F.Cu" "F.Mask" "F.Paste")
@@
 		)
 		(pad "SH" thru_hole oval
-			(at -4.32 -3)
+			(at -4.32 -3 90)
 			(size 1.1 1.7)
 			(drill oval 0.6 1.2)
@@
 		)
 		(pad "SH" thru_hole oval
-			(at -4.32 0.8)
+			(at -4.32 0.8 90)
 			(size 1.1 1.7)
 			(drill oval 0.6 1.2)
@@
 		)
 		(pad "SH" thru_hole oval
-			(at 4.32 -3)
+			(at 4.32 -3 90)
 			(size 1.1 1.7)
 			(drill oval 0.6 1.2)
@@
 		)
 		(pad "SH" thru_hole oval
-			(at 4.32 0.8)
+			(at 4.32 0.8 90)
 			(size 1.1 1.7)
 			(drill oval 0.6 1.2)
@@
 	(footprint "Resistor_SMD:R_0805_2012Metric"
 		(layer "F.Cu")
-		(at 135.655 118.175)
+		(at 142.38 121.66)
 		(descr "Resistor SMD 0805 (2012 Metric), square (rectangular) end terminal, IPC-7351 nominal, (Body size source: IPC-SM-782 page 72, https://www.pcb-3d.com/wordpress/wp-content/uploads/ipc-sm-782a_amendment_1_and_2.pdf)")
 		(tags "resistor")
@@
 	(footprint "Capacitor_SMD:C_0805_2012Metric"
 		(layer "F.Cu")
-		(at 131.225 115.315)
+		(at 137.95 118.8)
 		(descr "Capacitor SMD 0805 (2012 Metric), square (rectangular) end terminal, IPC-7351 nominal, (Body size source: IPC-SM-782 page 76, https://www.pcb-3d.com/wordpress/wp-content/uploads/ipc-sm-782a_amendment_1_and_2.pdf, https://docs.google.com/spreadsheets/d/1BsfQQcO9C6DZCsRaXUlFlo91Tg2WpOkGARC1WS5S8t0/edit?usp=sharing)")
 		(tags "capacitor")
@@
 		)
 	)
+	(gr_circle
+		(center 172 108.5)
+		(end 148.5 60)
+		(stroke
+			(width 0.2)
+			(type default)
+		)
+		(fill no)
+		(layer "F.Cu")
+		(net "/Call Next")
+	)
 	(embedded_fonts no)
